File: PhaseLatch.kicad_pcb (KiCad board)
At the start: 4 copper layers, 68.8 x 53.6 mm, 102 parts, among them J2 NC, J20 I_IN, J21 Q_IN, J23 CLK_IN, J5 Databus, J6 Chip select, J7 Addressbus, J8 Signals, P1 Conn_02x10_Odd_Even, P2 Conn_02x10_Odd_Even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

Commit message: Series termination, fork resistors
Parts:
- added R29: 33, Resistor_SMD:R_0402_1005Metric, F.Cu at (160.7, 121.2)
- added R30: 33, Resistor_SMD:R_0402_1005Metric, F.Cu at (160.7, 120.2)
- added R31: 33, Resistor_SMD:R_0402_1005Metric, F.Cu at (160.7, 119.2)
- added R32: 33, Resistor_SMD:R_0402_1005Metric, F.Cu at (160.7, 118.2)
- added R33: 33, Resistor_SMD:R_0402_1005Metric, F.Cu at (160.7, 117.3)
- added R34: 33, Resistor_SMD:R_0402_1005Metric, F.Cu at (160.7, 116.3)
- added R35: 33, Resistor_SMD:R_0402_1005Metric, F.Cu at (160.7, 115.4)
- added R36: 33, Resistor_SMD:R_0402_1005Metric, F.Cu at (160.7, 114.5)
- added R37: 33, Resistor_SMD:R_0402_1005Metric, F.Cu at (160.7, 113.7)
- added R38: 33, Resistor_SMD:R_0402_1005Metric, F.Cu at (160.7, 112.7)
- added R39: 10, Resistor_SMD:R_0402_1005Metric, F.Cu at (164.7, 119.2)
- added R40: 10, Resistor_SMD:R_0402_1005Metric, F.Cu at (164.7, 118.2)
- added R41: 10, Resistor_SMD:R_0402_1005Metric, F.Cu at (164.8, 117.2)
- added R42: 10, Resistor_SMD:R_0402_1005Metric, F.Cu at (164.8, 116.3)
- added R43: 10, Resistor_SMD:R_0402_1005Metric, F.Cu at (164.7, 115.3)
- added R44: 10, Resistor_SMD:R_0402_1005Metric, F.Cu at (164.8, 114.3)
- added R45: 10, Resistor_SMD:R_0402_1005Metric, F.Cu at (164.8, 113.4)
- added R46: 10, Resistor_SMD:R_0402_1005Metric, F.Cu at (164.8, 112.4)
- moved R13 21.7 mm to (187.1, 107.0)
- moved R12 15.3 mm to (172.5, 120.4), turned to -90 degrees
- moved R14 11.8 mm to (173.6, 120.4), turned to 90 degrees
- moved JP1 9.29 mm to (168.8, 110.5), turned to -90 degrees
- moved JP15 7.13 mm to (153.8, 117.0)
- moved R3 6.58 mm to (146.4, 122.2)
- moved R2 4.59 mm to (150.1, 110.7)
- moved JP10 2.82 mm to (157.2, 124.0)
- moved C22 1.87 mm to (152.7, 123.9)
- moved C24 1.52 mm to (159.2, 122.5)
- moved C23 1.15 mm to (161.3, 122.7)
- moved R8 1.06 mm to (183.8, 101.3), turned to 180 degrees
- moved C18 0.79 mm to (150.4, 124.2), turned to 180 degrees
- moved R18 0.63 mm to (176.2, 101.3), turned to 0 degrees
- moved R20 0.51 mm to (181.5, 101.3), turned to 180 degrees
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Connections:
- P1 pad 17: D7 -> /PB7
- P1 pad 18: D6 -> /PB6
- P1 pad 19: D5 -> /PB5
- P1 pad 20: D4 -> /PB4
- P2 pad 15: D0 -> /PB0
- P2 pad 16: D1 -> /PB1
- P2 pad 17: D2 -> /PB2
- P2 pad 18: D3 -> /PB3
- U1 pad 10: D5 -> Net-(U1-D7)
- U1 pad 11: D6 -> Net-(U1-D8)
- U1 pad 12: D7 -> Net-(U1-D9)
- U1 pad 3: /PD0 -> Net-(U1-D0)
- U1 pad 4: /PD1 -> Net-(U1-D1)
- U1 pad 5: D0 -> Net-(U1-D2)
- U1 pad 6: D1 -> Net-(U1-D3)
- U1 pad 7: D2 -> Net-(U1-D4)
- U1 pad 8: D3 -> Net-(U1-D5)
- U1 pad 9: D4 -> Net-(U1-D6)
Routing:
- net A0: track 0.00 -> 59.5 mm, vias 0 -> 2
- net A1: track 0.00 -> 57.1 mm, vias 0 -> 1
- net A3: track 0.00 -> 56.1 mm, vias 0 -> 1
- net A6: track 0.00 -> 55.3 mm, vias 0 -> 1
- net A2: track 0.00 -> 54.1 mm, vias 0 -> 1
- net A5: track 0.00 -> 53.7 mm
- net A4: track 0.00 -> 51.2 mm, vias 0 -> 1
- net A7: track 0.00 -> 48.4 mm, vias 0 -> 1
- net /"$0400": track 0.00 -> 44.4 mm, vias 0 -> 3
- net A9: track 0.00 -> 32.4 mm, vias 0 -> 1
- net A10: track 0.00 -> 30.2 mm, vias 0 -> 1
- net A11: track 0.00 -> 29.3 mm, vias 0 -> 1
- net A8: track 0.00 -> 27.6 mm, vias 0 -> 1
- net /PB4: track 0.00 -> 25.0 mm, vias 0 -> 1
- net /PB1: track 0.00 -> 24.7 mm, vias 0 -> 1
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
Commit message: Routing
Parts:
- moved R13 15.5 mm to (172.1, 103.1)
- moved U6 11.0 mm to (187.6, 103.8)
- moved C21 8.77 mm to (144.3, 109.5)
- moved JP1 7.53 mm to (161.4, 109.5)
- moved C17 4.73 mm to (147.4, 117.5)
- moved JP8 4.16 mm to (139.5, 112.3)
- moved C9 2.96 mm to (142.3, 120.0)
- moved C4 2.86 mm to (139.9, 120.7)
- moved C5 2.86 mm to (139.9, 119.7)
- moved R9 0.97 mm to (172.0, 135.6)
- moved R10 0.75 mm to (169.0, 135.6)
- moved JP5 0.70 mm to (165.6, 132.2)
- moved JP4 0.45 mm to (165.6, 134.5)
- moved R15 0.44 mm to (148.4, 113.0)
- moved JP9 0.20 mm to (143.5, 122.4)
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Routing:
- net /A13: track 0.00 -> 99.7 mm, vias 0 -> 5
- net /PHI0: track 0.00 -> 68.4 mm, vias 0 -> 2
- net /~{RW}: track 0.00 -> 63.9 mm, vias 0 -> 2
- net +Ext_3V3: track 0.00 -> 55.0 mm, vias 0 -> 2
- net /A14: track 0.00 -> 51.4 mm, vias 0 -> 1
- net Net-(U4-~{WE}): track 0.00 -> 28.7 mm, vias 0 -> 2
- net Net-(JP2-B): track 2.55 -> 16.9 mm, vias 0 -> 2
- net Net-(JP9-A): track 28.3 -> 15.5 mm
- net VCC: track 4.49 -> 17.1 mm, vias 2 -> 12
- net Net-(JP1-B): track 0.00 -> 9.55 mm, vias 0 -> 1
- net Net-(JP8-A): track 22.1 -> 15.4 mm
- net /FIFOADR1: track 0.00 -> 5.53 mm
- net Net-(U4-~{OE}): track 0.00 -> 5.51 mm
- net Net-(JP1-C): track 0.00 -> 5.26 mm
- net Net-(JP8-B): track 2.91 -> 6.72 mm
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Other:
- board text added: "CLK-In"
- board text added: "PhaseLatch"
- board text added: "v1.0"
- board text removed: "Aux (CLK2)"
- board text removed: "PhaseLatch v1.0"
