File: PhaseLatch.kicad_pcb (KiCad board)
At the start: 4 copper layers, 68.8 x 53.6 mm, 124 parts, among them J2 NC, J20 I_IN, J21 Q_IN, J23 CLK_IN, J5 Databus, J6 Chip select, J7 Addressbus, J8 Signals, P1 Conn_02x10_Odd_Even, P2 Conn_02x10_Odd_Even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

Commit message: IQ bias offset, IQ balancing, documentation
Parts:
- removed JP24, JP25: ~, Jumper:SolderJumper-2_P1.3mm_Bridged_RoundedPad1.0x1.5mm
- added C28: 620pF, Capacitor_SMD:C_0402_1005Metric, F.Cu at (131.9, 114.4)
- added C29: 330pF, Capacitor_SMD:C_0402_1005Metric, F.Cu at (135.5, 116.3)
- added C30: 330pF, Capacitor_SMD:C_0402_1005Metric, F.Cu at (128.2, 112.8)
- added C31: 330pF, Capacitor_SMD:C_0402_1005Metric, F.Cu at (128.2, 102.7)
- added C32: 620pF, Capacitor_SMD:C_0402_1005Metric, F.Cu at (132.0, 103.2)
- added C33: 330pF, Capacitor_SMD:C_0402_1005Metric, F.Cu at (135.5, 105.3)
- added FB2: FerriteBead_Small, Inductor_SMD:L_0603_1608Metric, F.Cu at (138.8, 100.0)
- added JP12: SolderJumper_2_Open, Jumper:SolderJumper-2_P1.3mm_Open_RoundedPad1.0x1.5mm, F.Cu at (145.8, 129.7)
- added JP28: ~, Jumper:SolderJumper-2_P1.3mm_Bridged_RoundedPad1.0x1.5mm, B.Cu at (151.5, 126.2)
- added L1: 1.2uH, Inductor_SMD:L_0603_1608Metric, F.Cu at (130.1, 113.3)
- added L2: 1.2uH, Inductor_SMD:L_0603_1608Metric, F.Cu at (133.7, 115.3)
- added L3: 1.2uH, Inductor_SMD:L_0603_1608Metric, F.Cu at (130.2, 102.0)
- added L4: 1.2uH, Inductor_SMD:L_0603_1608Metric, F.Cu at (133.7, 104.3)
- added R47: 33, Resistor_SMD:R_0402_1005Metric, F.Cu at (165.3, 132.2)
- added R48: 10k, Resistor_SMD:R_0402_1005Metric, F.Cu at (167.6, 93.7)
- added R49: 4k7, Resistor_SMD:R_0402_1005Metric, F.Cu at (134.4, 132.3)
- added R50: 4k7, Resistor_SMD:R_0402_1005Metric, F.Cu at (134.4, 130.4)
- added R51: 33, Resistor_SMD:R_0402_1005Metric, F.Cu at (131.0, 132.1)
- R15, R16: value NC -> 1k
- U1: value AD9201 -> HT9201ARSZ
- moved JP15 14.9 mm to (145.8, 129.7)
- moved C21 10.2 mm to (145.9, 117.9), turned to -90 degrees
- moved JP10 8.49 mm to (148.9, 126.2)
- moved C15 7.11 mm to (136.2, 106.6)
- moved C13 6.99 mm to (136.2, 117.6)
- moved T1 3.66 mm to (135.5, 110.8)
- moved JP6 3.66 mm to (137.8, 108.6)
- moved JP7 3.65 mm to (138.0, 119.4)
- moved T2 3.21 mm to (135.4, 121.6)
- moved C16 1.60 mm to (143.4, 117.8)
- moved C22 1.24 mm to (153.4, 123.0), turned to 0 degrees
- moved R1 0.94 mm to (144.0, 116.5)
- moved R3 0.84 mm to (146.4, 123.2)
- moved R26 0.76 mm to (141.3, 116.4)
- moved C1 0.60 mm to (133.0, 132.1)
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Connections:
- C1 pad 1: Net-(J23-In) -> Net-(C1-Pad1)
- C13 pad 2: Net-(J21-In) -> Net-(C13-Pad2)
- C15 pad 2: Net-(J20-In) -> Net-(C15-Pad2)
- JP19 pad 2: VCC -> Net-(JP19-C)
- JP4 pad 2: /IFCLK -> Net-(JP4-B)
- JP5 pad 2: /IFCLK -> Net-(JP4-B)
- U3 pad 6: Net-(JP25-B) -> VCC
- U3 pad 7: Net-(JP24-B) -> VCC
Routing:
- net Net-(JP1-B): track 8.92 -> 30.4 mm, vias 1 -> 2
- net Net-(JP15-A): track 24.2 -> 8.33 mm
- net Net-(JP10-A): track 7.32 -> 17.4 mm
- net Net-(JP19-C): track 0.00 -> 7.46 mm
- net Net-(U4-~{WE}): track 19.2 -> 13.3 mm
- net USRLED4: track 2.51 -> 7.53 mm
- net Net-(JP4-B): track 0.00 -> 4.65 mm, vias 0 -> 1
- net Net-(JP7-B): track 20.2 -> 15.8 mm
- net Net-(JP25-B): track 3.87 -> 0.00 mm
- net Net-(JP6-A): track 7.39 -> 3.59 mm
- net Net-(JP14-B): track 21.0 -> 17.4 mm
- net Net-(JP24-B): track 3.49 -> 0.00 mm
- net Net-(JP6-B): track 19.5 -> 16.0 mm
- net VCC: track 33.5 -> 36.9 mm
- net Net-(JP7-A): track 6.97 -> 4.06 mm
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Other:
- board text added: "CLKOUT"
- board text added: "IFCLK"
- board text added: "P1"
- board text added: "P2"
- board text added: "v1.2"
- board text removed: "v1.1"
